Commit message: Update vast_fake and modify vast_navigation

File: vast_gazebo/urdf/vast01_omni_practical.xacro (robot description, xacro)
@@ -144,5 +144,5 @@
 	</link>
 	<!-- IMU -->
-	<joint name="imu_sensor_joint" type="continuous">
+	<joint name="imu_sensor_joint" type="fixed">
         <axis xyz="0 0 1" />
         <origin xyz="-0.03 -0.12 0.32" rpy="0 0 0"/>
@@ -162,5 +162,5 @@
                 <box size="0.02 0.02 0.02"/>
             </geometry>
-            <material name="iRobot/Red"/>
+            <material name="blue"/>
         </visual>
         <inertial>
